Commit message: example.launch.pyを改善・mycobot_example.cppを変更

File: mycobot_280_description/urdf/mycobot_urdf.urdf (robot description, URDF)
Before this commit: robot mycobot_280, 7 links, 6 joints
Links:
- removed link base
- added link base_link; collision mesh filename=package://mycobot_280_description/meshes/mycobot_280/base.d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; visual mesh filename=package://mycobot_280_description/meshes/mycobot_280/base.d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
- link link1: geometry collision mesh filename=package://mycobot_280_description/meshes/mycobot_280/link1.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; visual mesh filename=package://mycobot_280_description/meshes/mycobot_280/link1.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
- link link2: geometry collision mesh filename=package://mycobot_280_description/meshes/mycobot_280/link2.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; visual mesh filename=package://mycobot_280_description/meshes/mycobot_280/link2.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
- link link3: geometry collision mesh filename=package://mycobot_280_description/meshes/mycobot_280/link3.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; visual mesh filename=package://mycobot_280_description/meshes/mycobot_280/link3.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
- link link4: geometry collision mesh filename=package://mycobot_280_description/meshes/mycobot_280/link4.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; visual mesh filename=package://mycobot_280_description/meshes/mycobot_280/link4.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
- link link5: geometry collision mesh filename=package://mycobot_280_description/meshes/mycobot_280/link5.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; visual mesh filename=package://mycobot_280_description/meshes/mycobot_280/link5.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
- link link6: geometry collision mesh filename=package://mycobot_280_description/meshes/mycobot_280/link6.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; visual mesh filename=package://mycobot_280_description/meshes/mycobot_280/link6.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
Joints:
- joint joint1: parent base -> base_link
